Commit message: fix lidar and controllers

File: urdf/car_fix_wheels.urdf (robot description, URDF)
Before this commit: robot car_fix_wheels, 9 links, 8 joints
Joints:
- joint lidar_joint: origin xyz=0.3 0 0.07 rpy=0 0 0 -> xyz=0.4 0 0.07 rpy=0 0 0

Commit message: commit

File: urdf/car_fix_wheels.urdf (robot description, URDF)
Before this commit: robot car_fix_wheels, 9 links, 8 joints
Links:
- added link imu_link, mass 0.01; visual box size=0.01 0.01 0.01
Joints:
- added joint imu_joint: type fixed, parent base_link, child imu_link, origin xyz=0 0 0.1 rpy=0 0 0
